File: AirMonitor.kicad_sch (KiCad schematic)
At the start: 60 parts, among them J1 Conn_01x03, J3 USB_C_Receptacle_USB2.0, SW1 RST, SW2 BOOT, U1 WS2812B-2020, U10 AZ1117-3V3, U2 BMP581, U3 SHT45, U4 SCD41, U5 PMS7003, U6 SGP41, U7 5V5, U8 AZ1117-3V3, U9 ESP32-C3-MINI-1

Commit message: Working revision
Parts:
- J1: MPN (none) -> NO_MPN
- U9: MPN (none) -> ESP32-C3-MINI-1-N4; Mouser (none) -> 356-ESP32-C3-MINI1N4
Other:
- company: (none) -> Jakub Jendryka
- title: (none) -> AirMonitor
Changed lines of the file:
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@@
 (kicad_sch (version 20230121) (generator eeschema)
   (paper "A3")
+  (title_block
+    (title "AirMonitor")
+    (date "2023-12-09")
+    (rev "1.0.0")
+    (company "Jakub Jendryka")
+  )
   (bus_alias "I2C" (members "SDA" "SCL"))
   (bus_alias "JTAG" (members "TCK" "TDI" "TDO" "TMS"))
@@
     )
     (property "Datasheet" "https://www.espressif.com/sites/default/files/documentation/esp32-c3-mini-1_datasheet_en.pdf" (at 173.99 173.99 0)
+      (effects (font (size 1.27 1.27)) hide)
+    )
+    (property "MPN" "ESP32-C3-MINI-1-N4" (at 173.99 135.89 0)
+      (effects (font (size 1.27 1.27)) hide)
+    )
+    (property "Mouser" "356-ESP32-C3-MINI1N4" (at 173.99 135.89 0)
       (effects (font (size 1.27 1.27)) hide)
     )
@@
       (effects (font (size 1.27 1.27)) hide)
     )
+    (property "MPN" "NO_MPN" (at 217.17 114.3 0)
+      (effects (font (size 1.27 1.27)) hide)
+    )
